File: GearTest/GearTest.kicad_pcb (KiCad board)
At the start: 2 copper layers, 71.4 x 55.6 mm, 8 parts, among them J1 Jack-DC, J2 Conn_01x02_Socket, M1 Motor_DC, M2 Motor_DC, Q1 IRLZ44N, U1 WeAct BlackPill STM32F411C_C-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, U2 INA219

Commit message: dev
Parts:
- removed J1: Jack-DC, Connector_Wire:SolderWire-0.5sqmm_1x02_P4.8mm_D0.9mm_OD2.3mm
- added SW3: SW_Push, Button_Switch_THT:SW_CK_JS202011CQN_DPDT_Straight, F.Cu at (157.2, 76.1)
Connections:
- J2 pad 2: Net-(J2-Pin_2) -> GND
- M1 pad 1: 12V0 -> Net-(M1-+)
- M2 pad 1: Net-(J2-Pin_1) -> Net-(M2-+)
- U1 pad 3: /MOTOR_GATE -> unconnected-(U1-PC14-Pad3)
- U1 pad 31: unconnected-(U1-PA10-Pad31) -> Net-(U1-PA10)
- U1 pad 33: unconnected-(U1-PA12-Pad33) -> /MOTOR_GATE
- U1 pad 42: unconnected-(U1-PB6-Pad42) -> /END_MOTOR_SCL
- U1 pad 43: unconnected-(U1-PB7-Pad43) -> /END_MOTOR_SDA
- U1 pad 45: /END_MOTOR_SCL -> unconnected-(U1-PB8-Pad45)
- U1 pad 46: /END_MOTOR_SDA -> unconnected-(U1-PB9-Pad46)
- U2 pad 5: GND -> Net-(J2-Pin_1)
- U2 pad 6: Net-(J2-Pin_2) -> Net-(M2-+)
- U2 pad VIN+: Net-(J2-Pin_2) -> Net-(M2-+)
- U2 pad VIN-: GND -> Net-(J2-Pin_1)
Routing:
- net 12V0: track 20.9 -> 0.28 mm
- net /MOTOR_GATE: track 19.1 -> 0.00 mm
- net Net-(J2-Pin_2): track 16.3 -> 0.00 mm
- net Net-(J2-Pin_1): track 10.6 -> 1.27 mm
- net Net-(M1--): track 7.09 -> 0.00 mm
- net /END_MOTOR_SDA: track 9.60 -> 11.7 mm
- net /END_MOTOR_SCL: track 9.60 -> 11.6 mm
- net Net-(M2-+): track 0.00 -> 1.98 mm
- net Net-(M1-+): track 0.00 -> 0.57 mm
Other:
- board size 71.4 x 55.6 mm -> 80 x 80 mm

Commit message: dev
Parts:
- removed DC1: Mini 560 Step-down, Footprints:MINI 560 PRO
- added C1: 0.1u, Capacitor_SMD:C_0805_2012Metric_Pad1.18x1.45mm_HandSolder, B.Cu at (97.6, 152.7)
- added C2: 0.1u, Capacitor_SMD:C_0805_2012Metric_Pad1.18x1.45mm_HandSolder, B.Cu at (134.5, 80.9)
- added C3: 1000u 35М, Capacitor_THT:CP_Radial_D13.0mm_P5.00mm, F.Cu at (128.5, 90.9)
- added D1: ~, Footprints:WeAct DCM1 LGS5148, B.Cu at (84.0, 72.3)
- added D2: ~, Footprints:WeAct DCM1 LGS5148, B.Cu at (97.9, 87.0)
- added J3: Терминал выключателя основного питания, TerminalBlock_Phoenix:TerminalBlock_Phoenix_MPT-0,5-5-2.54_1x05_P2.54mm_Horizontal, F.Cu at (117.2, 52.6)
- added J5: Терминал питания XY-FZ35, TerminalBlock_Phoenix:TerminalBlock_Phoenix_MPT-0,5-2-2.54_1x02_P2.54mm_Horizontal, F.Cu at (106.9, 64.6)
- added J6: Терминал LCD_1602_I2C, TerminalBlock_Phoenix:TerminalBlock_Phoenix_MPT-0,5-4-2.54_1x04_P2.54mm_Horizontal, F.Cu at (103.8, 109.3)
- added J7: Терминал UART1, TerminalBlock_Phoenix:TerminalBlock_Phoenix_MPT-0,5-5-2.54_1x05_P2.54mm_Horizontal, F.Cu at (116.4, 146.4)
- added R2: 10k, Resistor_SMD:R_0603_1608Metric_Pad0.98x0.95mm_HandSolder, B.Cu at (97.3, 147.7)
- added R3: 5.1k, Resistor_SMD:R_0603_1608Metric_Pad0.98x0.95mm_HandSolder, B.Cu at (124.0, 154.3)
- added R4: 5.1k, Resistor_SMD:R_0603_1608Metric_Pad0.98x0.95mm_HandSolder, B.Cu at (126.5, 154.3)
- added SW1: Выключатель моторов, TerminalBlock_Phoenix:TerminalBlock_Phoenix_MPT-0,5-3-2.54_1x03_P2.54mm_Horizontal, F.Cu at (95.7, 65.8)
- added U2: CH340N, Package_SO:JEITA_SOIC-8_3.9x4.9mm_P1.27mm, B.Cu at (108.2, 146.3)
- J2: value Conn_01x02_Socket -> Терминал выключателя моторов; footprint Connector_Wire:SolderWire-0.5sqmm_1x02_P4.8mm_D0.9mm_OD2.3mm -> TerminalBlock_Phoenix:TerminalBlock_Phoenix_MPT-0,5-5-2.54_1x05_P2.54mm_Horizontal
- M1, M2: footprint Connector_Wire:SolderWire-0.75sqmm_1x02_P7mm_D1.25mm_OD3.5mm -> TerminalBlock_Phoenix:TerminalBlock_Phoenix_MPT-0,5-2-2.54_1x02_P2.54mm_Horizontal
- SW3: footprint Button_Switch_THT:SW_CK_JS202011CQN_DPDT_Straight -> TerminalBlock_Phoenix:TerminalBlock_Phoenix_MPT-0,5-2-2.54_1x02_P2.54mm_Horizontal
- moved SW3 97.1 mm to (91.5, 147.7), turned to 180 degrees
- moved U1 50.6 mm to (107.5, 128.3), turned to 0 degrees
- moved J2 41.1 mm to (102.4, 52.6), turned to 0 degrees
- moved M2 36.6 mm to (132.0, 52.6), turned to 0 degrees
- moved M1 23.5 mm to (95.0, 52.6), turned to 0 degrees
- moved U3 9.77 mm to (124.5, 72.4), turned to 0 degrees
- moved Q1 3.88 mm to (82.4, 54.6), turned to 0 degrees
- renumbered U2 to U3
Connections:
- J2 pad 1: Net-(J2-Pin_1) -> 12V0
- J2 pad 2: GND -> Net-(J2-Pin_2)
- M1 pad 1: Net-(M1-+) -> Net-(J2-Pin_2)
- M2 pad 2: GND -> GNDPWR
- Q1 pad 3: GND -> GNDPWR
- SW3 pad 1: Net-(U1-PA10) -> Net-(U1-PA9)
- SW3 pad 2: GND -> GNDD
- U1 pad 29: unconnected-(U1-PA8-Pad29) -> /LCD1602_MOTOR_SCL
- U1 pad 30: unconnected-(U1-PA9-Pad30) -> Net-(U1-PA9)
- U1 pad 31: Net-(U1-PA10) -> /UART1_RX
- U1 pad 40: unconnected-(U1-PB4-Pad40) -> /LCD1602_MOTOR_SDA
- U1 pad 42: /END_MOTOR_SCL -> /UART1_TX
- U1 pad 43: /END_MOTOR_SDA -> unconnected-(U1-PB7-Pad43)
- U1 pad 45: unconnected-(U1-PB8-Pad45) -> /INA219_MOTOR_SCL
- U1 pad 46: unconnected-(U1-PB9-Pad46) -> /INA219_MOTOR_SDA
- U3 pad 2: GND -> GNDD
- U3 pad 3: /END_MOTOR_SDA -> /INA219_MOTOR_SDA
- U3 pad 4: /END_MOTOR_SCL -> /INA219_MOTOR_SCL
- U3 pad 5: Net-(J2-Pin_1) -> Net-(U3-PadVIN-)
Routing:
- net 12V0: track 0.28 -> 107.6 mm
- net 3V3: track 82.2 -> 167.4 mm
- net /LCD1602_MOTOR_SCL: track 0.00 -> 82.3 mm
- net /LCD1602_MOTOR_SDA: track 0.00 -> 79.5 mm
- net 5V0: track 0.00 -> 62.8 mm
- net /INA219_MOTOR_SCL: track 0.00 -> 40.8 mm
- net GNDD: track 0.00 -> 39.1 mm
- net /INA219_MOTOR_SDA: track 0.00 -> 36.9 mm
- net Net-(J2-Pin_2): track 0.00 -> 27.9 mm
- net Net-(U1-PA9): track 0.00 -> 25.5 mm
- net Net-(M1--): track 0.00 -> 21.0 mm
- net Net-(M2-+): track 1.98 -> 19.5 mm
- net /USB_D-: track 0.00 -> 15.2 mm
- net /UART1_RX: track 0.00 -> 14.3 mm
- net /USB_D+: track 0.00 -> 13.9 mm
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- added copper zone on B.Cu, net GNDD
- added copper zone on B.Cu, net GNDPWR
- removed copper zone on F.Cu, net GND
Other:
- board size 80 x 80 mm -> 62.4 x 113 mm

Commit message: dev
Parts:
- removed SW1: Выключатель моторов, TerminalBlock_Phoenix:TerminalBlock_Phoenix_MPT-0,5-3-2.54_1x03_P2.54mm_Horizontal
- added D1: SS34, Diode_SMD:D_SMA, B.Cu at (97.7, 53.7)
- added D2: SS34, Diode_SMD:D_SMA, B.Cu at (134.7, 61.2)
- added H1: MountingHole, MountingHole:MountingHole_2.2mm_M2_DIN965_Pad_TopOnly, B.Cu at (74.7, 135.2)
- added H2: MountingHole, MountingHole:MountingHole_2.2mm_M2_DIN965_Pad_TopOnly, B.Cu at (140.7, 135.2)
- added H3: MountingHole, MountingHole:MountingHole_2.2mm_M2_DIN965_Pad_TopOnly, B.Cu at (74.7, 50.2)
- added R1: 0R, Resistor_SMD:R_2512_6332Metric_Pad1.40x3.35mm_HandSolder, B.Cu at (135.9, 99.9)
- added R2: 0R, Resistor_SMD:R_2512_6332Metric_Pad1.40x3.35mm_HandSolder, B.Cu at (140.2, 77.2)
- added R3: 0R, Resistor_SMD:R_2512_6332Metric_Pad1.40x3.35mm_HandSolder, B.Cu at (117.0, 67.6)
- added R4: 10k, Resistor_SMD:R_0603_1608Metric_Pad0.98x0.95mm_HandSolder, B.Cu at (104.7, 64.7)
- J2: footprint TerminalBlock_Phoenix:TerminalBlock_Phoenix_MPT-0,5-5-2.54_1x05_P2.54mm_Horizontal -> TerminalBlock_Phoenix:TerminalBlock_Phoenix_MPT-0,5-3-2.54_1x03_P2.54mm_Horizontal
- moved J5 30.0 mm to (91.0, 82.2), turned to -90 degrees
- moved R6 28.4 mm to (129.1, 126.4), turned to 0 degrees
- moved R7 28.1 mm to (123.3, 126.4), turned to 0 degrees
- moved J7 20.9 mm to (131.0, 131.5), turned to 180 degrees
- moved C1 19.6 mm to (87.1, 136.1), turned to -90 degrees
- moved Q1 19.6 mm to (99.2, 64.6), turned to 90 degrees
- moved SW3 19.1 mm to (87.1, 129.1), turned to 90 degrees
- moved U2 15.1 mm to (109.6, 131.3)
- moved U1 15.1 mm to (108.9, 113.2)
- moved R5 13.1 mm to (91.1, 136.1), turned to -90 degrees
- moved J6 8.14 mm to (105.4, 72.6)
- moved D4 6.55 mm to (104.5, 87.0)
- moved C2 6.54 mm to (130.0, 76.1), turned to 180 degrees
- moved M1 6.26 mm to (88.7, 52.7)
- moved J2 3.82 mm to (106.2, 52.6)
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- renumbered D1 to D3, D2 to D4, J6 to J5, J5 to J6, R2 to R5, R3 to R6, R4 to R7
Connections:
- net Net-(U3-PadVIN-) renamed /L+
- J2 pad 2: Net-(J2-Pin_2) -> Net-(D1-A)
- J2 pad 3: Net-(J2-Pin_2) -> GNDPWR
- J5 pad 1: GNDD -> GNDPWR
- J6 pad 2: GNDD -> GNDPWR
- M1 pad 1: Net-(J2-Pin_2) -> Net-(D1-A)
- Q1 pad 1: /MOTOR_GATE -> Net-(Q1-G)
- U1 pad 11: unconnected-(U1-PA1-Pad11) -> /MOTOR_GATE
- U1 pad 33: /MOTOR_GATE -> unconnected-(U1-PA12-Pad33)
Routing:
- net /INA219_MOTOR_SCL: track 40.8 -> 121.5 mm
- net /INA219_MOTOR_SDA: track 36.9 -> 115.2 mm
- net Net-(R2-Pad2): track 0.00 -> 62.4 mm
- net 5V0: track 62.8 -> 16.6 mm
- net 12V0: track 107.6 -> 149.6 mm
- net Net-(D2-K): track 19.5 -> 61.3 mm
- net Net-(D1-A): track 0.00 -> 34.4 mm
- net GNDD: track 39.1 -> 8.10 mm
- net Net-(J2-Pin_2): track 27.9 -> 0.00 mm
- net /LCD1602_MOTOR_SCL: track 82.3 -> 54.6 mm
- net Net-(Q1-G): track 0.00 -> 21.6 mm
- net Net-(R1-Pad2): track 0.00 -> 20.2 mm
- net /MOTOR_GATE: track 0.00 -> 18.9 mm
- net GNDPWR: track 9.38 -> 24.4 mm
- net /USB_D-: track 15.2 -> 23.3 mm
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- added copper zone on B.Cu, net 12V0
Other:
- board size 62.4 x 113 mm -> 76 x 95 mm
